File: Poop-Valve/Poop-Valve.sch (KiCad schematic (older format))
At the start: 39 parts

Commit message: v0.6 fix led connector pinout
Parts:
- added J?: Ovr Sw, symbol Connector:Conn_01x05_Male
Connections:
- wire segments 243 -> 249
- no-connect marks 9 -> 10
Other:
- note added: "Inline"
- moved on the sheet: J?
Changed lines of the file:
@@
 P 1200 4400
 F 0 "SW?" H 1000 4200 50  0001 C CNN
-F 1 "Manual Override" H 1250 5000 50  0000 C CNN
+F 1 "Manual Override" H 1400 4200 50  0000 C CNN
 F 2 "" H 1200 4400 50  0001 C CNN
 F 3 "~" H 1200 4400 50  0001 C CNN
@@
 U 1 1 63AD73BF
 P 1200 4000
-F 0 "SW?" H 1050 4100 50  0000 C CNN
+F 0 "SW?" H 1400 4200 50  0000 C CNN
 F 1 "SW_DPDT_x2" H 1550 3950 50  0001 C CNN
 F 2 "" H 1200 4000 50  0001 C CNN
@@
 Wire Wire Line
 	1000 4500 650  4500
-Wire Wire Line
-	1400 4000 1550 4000
 Wire Notes Line
 	1200 3950 1200 4350
@@
 Wire Wire Line
 	1750 4000 2000 4000
-Connection ~ 1750 4400
 Wire Wire Line
 	1750 4400 2000 4400
 Wire Wire Line
-	1400 4400 1750 4400
+	1400 4400 1500 4400
 $Comp
 L Switch:SW_SPDT_MSM SW?
@@
 L power:GND #PWR?
 U 1 1 64417A2C
-P 900 2750
-F 0 "#PWR?" H 900 2500 50  0001 C CNN
-F 1 "GND" H 905 2577 50  0000 C CNN
-F 2 "" H 900 2750 50  0001 C CNN
-F 3 "" H 900 2750 50  0001 C CNN
-	1    900  2750
-	1    0    0    -1
-$EndComp
-$Comp
-L power:+3.3V #PWR?
-U 1 1 64418208
-P 1200 2750
-F 0 "#PWR?" H 1200 2600 50  0001 C CNN
-F 1 "+3.3V" H 1215 2923 50  0000 C CNN
-F 2 "" H 1200 2750 50  0001 C CNN
-F 3 "" H 1200 2750 50  0001 C CNN
-	1    1200 2750
+P 2200 2850
+F 0 "#PWR?" H 2200 2600 50  0001 C CNN
+F 1 "GND" H 2205 2677 50  0000 C CNN
+F 2 "" H 2200 2850 50  0001 C CNN
+F 3 "" H 2200 2850 50  0001 C CNN
+	1    2200 2850
 	1    0    0    -1
 $EndComp
@@
 L Connector:Conn_01x03_Male J?
 U 1 1 645F382F
-P 1200 3150
-F 0 "J?" V 1354 2962 50  0000 R CNN
-F 1 "Override" V 1263 2962 50  0000 R CNN
-F 2 "" H 1200 3150 50  0001 C CNN
-F 3 "~" H 1200 3150 50  0001 C CNN
-	1    1200 3150
-	0    -1   -1   0
+P 1800 2700
+F 0 "J?" H 2000 2500 50  0000 R CNN
+F 1 "Override" H 1950 2950 50  0000 R CNN
+F 2 "" H 1800 2700 50  0001 C CNN
+F 3 "~" H 1800 2700 50  0001 C CNN
+	1    1800 2700
+	1    0    0    -1
 $EndComp
 $Comp
@@
 Wire Wire Line
 	3300 4400 3300 2250
-Wire Wire Line
-	750  4100 750  3600
-Wire Wire Line
-	750  3600 1200 3600
-Wire Wire Line
-	1200 3600 1200 2950
 Connection ~ 750  4100
-Wire Wire Line
-	1200 2950 1200 2750
-Connection ~ 1200 2950
-Wire Wire Line
-	650  3900 650  3500
-Wire Wire Line
-	650  3500 1100 3500
-Wire Wire Line
-	1100 3500 1100 2950
 Connection ~ 650  3900
-Wire Wire Line
-	1100 2700 900  2700
-Wire Wire Line
-	900  2700 900  2750
-Wire Wire Line
-	1100 2700 1100 2950
-Connection ~ 1100 2950
-Wire Wire Line
-	1300 2950 1300 3500
-Wire Wire Line
-	1300 3500 1550 3500
-Wire Wire Line
-	1550 3500 1550 4000
-Wire Wire Line
-	1300 2800 1300 2950
-Wire Wire Line
-	1300 2800 3850 2800
-Connection ~ 1300 2950
 Wire Wire Line
 	7300 750  7300 850
@@
 Wire Wire Line
 	6400 1150 7000 1150
+Connection ~ 2000 2800
+Wire Wire Line
+	2000 2800 3850 2800
+Connection ~ 2000 2700
+Connection ~ 2000 2600
+$Comp
+L power:+3.3V #PWR?
+U 1 1 64418208
+P 2300 2700
+F 0 "#PWR?" H 2300 2550 50  0001 C CNN
+F 1 "+3.3V" H 2315 2873 50  0000 C CNN
+F 2 "" H 2300 2700 50  0001 C CNN
+F 3 "" H 2300 2700 50  0001 C CNN
+	1    2300 2700
+	1    0    0    -1
+$EndComp
+Wire Wire Line
+	2000 2700 2300 2700
+Wire Wire Line
+	2200 2850 2200 2600
+Wire Wire Line
+	2100 2600 2000 2600
+Wire Wire Line
+	2000 2600 2200 2600
+$Comp
+L Connector:Conn_01x05_Male J?
+U 1 1 636591C4
+P 850 3100
+F 0 "J?" V 912 2812 50  0000 R CNN
+F 1 "Ovr Sw" V 1003 2812 50  0000 R CNN
+F 2 "" H 850 3100 50  0001 C CNN
+F 3 "~" H 850 3100 50  0001 C CNN
+	1    850  3100
+	0    -1   1    0
+$EndComp
+Connection ~ 1750 4000
+Wire Wire Line
+	650  2600 650  3300
+Wire Wire Line
+	650  2600 2000 2600
+Connection ~ 650  3300
+Wire Wire Line
+	650  3300 650  3900
+Wire Wire Line
+	750  2700 750  3300
+Wire Wire Line
+	750  2700 2000 2700
+Connection ~ 750  3300
+Wire Wire Line
+	850  2800 850  3300
+Wire Wire Line
+	850  2800 2000 2800
+Wire Wire Line
+	750  3300 750  4100
+Connection ~ 850  3300
+Wire Wire Line
+	1400 4000 1400 3700
+Wire Wire Line
+	850  3700 1400 3700
+Wire Wire Line
+	850  3300 850  3700
+Wire Wire Line
+	1050 3300 1050 3600
+Wire Wire Line
+	1050 3600 1500 3600
+Wire Wire Line
+	1500 3600 1500 4400
+Connection ~ 1050 3300
+NoConn ~ 950  3300
+Text Notes 1150 3400 0    50   ~ 0
+Inline
+Wire Wire Line
+	1050 2900 1750 2900
+Wire Wire Line
+	1050 2900 1050 3300
+Wire Wire Line
+	1750 2900 1750 4000
 $EndSCHEMATC

Commit message: v0.7 correct ADC sample wiring
Parts:
- removed J?: V Sample, symbol Connector:Conn_01x02_Male
- added D?: Heart, symbol Device:LED
- added F?: 1A, symbol Device:Fuse_Small
- added J?: Sensor, symbol Connector:Conn_Coaxial_Power
- added J?: 24VDC, symbol Connector:Conn_Coaxial_Power
- added R?: 470, symbol Device:R
- added R?: 500/2W, symbol Device:R
- J?: value Ovr Sw -> Ovr Switch
Connections:
- wire segments 249 -> 256
Other:
- note added: "5.5x2.1"
- note added: "Inline (F)"
- note added: "Phono"
- note removed: "Inline"
- moved on the sheet: BT?, F?, J?
Changed lines of the file:
@@
 Sheet 1 1
 Title "Poop Valve Controller"
-Date "2022-10-19"
-Rev "0.6 (draft)"
+Date "2023-01-12"
+Rev "0.7 (draft)"
 Comp "Robert Ferguson Observatory"
-Comment1 "v0.6 fix led connector pinout"
+Comment1 "v0.4 fix override logic; detect override; resize"
 Comment2 "v0.5 add connectors"
-Comment3 "v0.4 fix override logic; detect override; resize"
-Comment4 "v0.3 pivot to manual override relay"
+Comment3 "v0.6 fix led connector pinout"
+Comment4 "v0.7 correct ADC sample wiring"
 $EndDescr
 $Comp
@@
 L Device:Battery BT?
 U 1 1 632C7943
-P 1500 6600
-F 0 "BT?" H 1500 6200 50  0000 C CNN
-F 1 "12V" H 1500 6300 50  0000 C CNN
-F 2 "" V 1500 6660 50  0001 C CNN
-F 3 "~" V 1500 6660 50  0001 C CNN
-	1    1500 6600
+P 1300 7550
+F 0 "BT?" H 1300 7150 50  0000 C CNN
+F 1 "12V" H 1300 7250 50  0000 C CNN
+F 2 "" V 1300 7610 50  0001 C CNN
+F 3 "~" V 1300 7610 50  0001 C CNN
+	1    1300 7550
 	1    0    0    -1
 $EndComp
@@
 L Connector:Conn_Coaxial_Power J?
 U 1 1 632E443C
-P 950 6550
-F 0 "J?" H 950 6100 50  0000 C CNN
-F 1 "Charger" H 950 6200 50  0000 C CNN
-F 2 "" H 950 6500 50  0001 C CNN
-F 3 "~" H 950 6500 50  0001 C CNN
-	1    950  6550
+P 750 7500
+F 0 "J?" H 750 7050 50  0000 C CNN
+F 1 "Charger" H 750 7150 50  0000 C CNN
+F 2 "" H 750 7450 50  0001 C CNN
+F 3 "~" H 750 7450 50  0001 C CNN
+	1    750  7500
 	1    0    0    -1
 $EndComp
@@
 	1    9050 5200
 	0    1    -1   0
-$EndComp
-$Comp
-L Connector:Conn_01x02_Male J?
-U 1 1 6362E2EC
-P 10300 5950
-F 0 "J?" H 10350 6100 50  0000 R CNN
-F 1 "V Sample" H 10600 5750 50  0000 R CNN
-F 2 "" H 10300 5950 50  0001 C CNN
-F 3 "~" H 10300 5950 50  0001 C CNN
-	1    10300 5950
-	-1   0    0    -1
 $EndComp
 $Comp
@@
 L Device:Fuse_Small F?
 U 1 1 63320CD5
-P 2350 6400
-F 0 "F?" H 2350 6585 50  0000 C CNN
-F 1 "1A" H 2350 6494 50  0000 C CNN
-F 2 "" H 2350 6400 50  0001 C CNN
-F 3 "~" H 2350 6400 50  0001 C CNN
-	1    2350 6400
-	1    0    0    -1
-$EndComp
-Wire Wire Line
-	950  6450 950  6400
-Wire Wire Line
-	950  6400 1500 6400
-Connection ~ 1500 6400
-Wire Wire Line
-	950  6750 950  6800
-Wire Wire Line
-	950  6800 1500 6800
-Wire Wire Line
-	1500 6800 1950 6800
-Connection ~ 1500 6800
+P 2150 6400
+F 0 "F?" H 2150 6585 50  0000 C CNN
+F 1 "1A" H 2150 6494 50  0000 C CNN
+F 2 "" H 2150 6400 50  0001 C CNN
+F 3 "~" H 2150 6400 50  0001 C CNN
+	1    2150 6400
+	1    0    0    -1
+$EndComp
+Wire Wire Line
+	750  7400 750  7350
+Wire Wire Line
+	750  7350 1300 7350
+Connection ~ 1300 7350
+Wire Wire Line
+	750  7700 750  7750
+Wire Wire Line
+	750  7750 1300 7750
+Wire Wire Line
+	1300 7750 1750 7750
+Connection ~ 1300 7750
 Text Notes 6300 3700 0    50   ~ 0
 * Open-Close
@@
 Wire Wire Line
 	3850 5750 4250 5750
-Text Notes 6200 4100 0    50   ~ 0
+Text Notes 6150 4000 0    50   ~ 0
 * GPIO26 logic:\n  Open is high\n  Close is low
 Wire Wire Line
@@
 	9700 5300 9550 5300
 Connection ~ 9700 5000
-Wire Wire Line
-	9350 5800 9350 5950
-Wire Wire Line
-	8400 6050 8400 5300
-Wire Wire Line
-	8400 5300 8450 5300
 $Comp
 L power:+12V #PWR?
@@
 Wire Wire Line
 	9150 3600 9150 4600
-Wire Wire Line
-	9350 5950 10100 5950
-Wire Wire Line
-	8400 6050 10100 6050
 Connection ~ 3850 2800
 Wire Wire Line
@@
 L Connector:Conn_Coaxial_Power J?
 U 1 1 63C43814
-P 2200 6550
-F 0 "J?" H 2200 6050 50  0000 C CNN
-F 1 "12VDC" H 2200 6150 50  0000 C CNN
-F 2 "" H 2200 6500 50  0001 C CNN
-F 3 "~" H 2200 6500 50  0001 C CNN
-	1    2200 6550
+P 1900 6550
+F 0 "J?" H 1650 6500 50  0000 C CNN
+F 1 "12VDC" H 1650 6400 50  0000 C CNN
+F 2 "" H 1900 6500 50  0001 C CNN
+F 3 "~" H 1900 6500 50  0001 C CNN
+	1    1900 6550
 	1    0    0    -1
 $EndComp
@@
 L Connector:Conn_Coaxial_Power J?
 U 1 1 63C5326A
-P 1950 6550
-F 0 "J?" V 2175 6500 50  0000 C CNN
-F 1 "Power" H 1900 6150 50  0000 C CNN
-F 2 "" H 1950 6500 50  0001 C CNN
-F 3 "~" H 1950 6500 50  0001 C CNN
-	1    1950 6550
-	1    0    0    -1
-$EndComp
-Wire Wire Line
-	1950 6400 1950 6450
-Wire Wire Line
-	1500 6400 1950 6400
-Wire Wire Line
-	1950 6800 1950 6750
+P 1750 7500
+F 0 "J?" V 1975 7450 50  0000 C CNN
+F 1 "Power" H 1700 7100 50  0000 C CNN
+F 2 "" H 1750 7450 50  0001 C CNN
+F 3 "~" H 1750 7450 50  0001 C CNN
+	1    1750 7500
+	1    0    0    -1
+$EndComp
+Wire Wire Line
+	1750 7350 1750 7400
+Wire Wire Line
+	1300 7350 1750 7350
+Wire Wire Line
+	1750 7750 1750 7700
 $Comp
 L Connector:Conn_01x02_Male J?
@@
 $EndComp
 Wire Wire Line
-	2200 6800 2200 6750
-Wire Wire Line
-	2200 6450 2200 6400
-Wire Wire Line
-	2200 6400 2250 6400
+	1900 6800 1900 6750
+Wire Wire Line
+	1900 6450 1900 6400
 Wire Wire Line
 	3850 5750 3850 6650
@@
 	3850 5550 3850 5750
 Wire Wire Line
-	2450 6400 2500 6400
-Wire Wire Line
-	2200 6800 2500 6800
-Wire Wire Line
 	2500 6400 2500 6550
 Connection ~ 2500 6400
 Wire Wire Line
 	2500 6650 2500 6800
-Connection ~ 2500 6800
 Wire Wire Line
 	3000 6550 3250 6550
@@
 P 850 3100
 F 0 "J?" V 912 2812 50  0000 R CNN
-F 1 "Ovr Sw" V 1003 2812 50  0000 R CNN
+F 1 "Ovr Switch" V 1003 2812 50  0000 R CNN
 F 2 "" H 850 3100 50  0001 C CNN
 F 3 "~" H 850 3100 50  0001 C CNN
@@
 NoConn ~ 950  3300
 Text Notes 1150 3400 0    50   ~ 0
-Inline
+Inline (F)
 Wire Wire Line
 	1050 2900 1750 2900
@@
 Wire Wire Line
 	1750 2900 1750 4000
+$Comp
+L Device:LED D?
+U 1 1 63AE6C12
+P 6800 4200
+F 0 "D?" V 6850 4400 50  0000 R CNN
+F 1 "Heart" V 6750 4500 50  0000 R CNN
+F 2 "" H 6800 4200 50  0001 C CNN
+F 3 "~" H 6800 4200 50  0001 C CNN
+	1    6800 4200
+	0    -1   -1   0
+$EndComp
+$Comp
+L Device:R R?
+U 1 1 63B22253
+P 6800 4500
+F 0 "R?" H 6650 4550 50  0000 L CNN
+F 1 "470" V 6800 4450 50  0000 L CNN
+F 2 "" V 6730 4500 50  0001 C CNN
+F 3 "~" H 6800 4500 50  0001 C CNN
+	1    6800 4500
+	1    0    0    -1
+$EndComp
+Wire Wire Line
+	6800 3800 6850 3800
+$Comp
+L power:GND #PWR?
+U 1 1 63B37882
+P 6800 4650
+F 0 "#PWR?" H 6800 4400 50  0001 C CNN
+F 1 "GND" H 6805 4477 50  0000 C CNN
+F 2 "" H 6800 4650 50  0001 C CNN
+F 3 "" H 6800 4650 50  0001 C CNN
+	1    6800 4650
+	1    0    0    -1
+$EndComp
+Wire Wire Line
+	6800 4050 6800 3800
+$Comp
+L Device:R R?
+U 1 1 63D72259
+P 8950 6150
+F 0 "R?" V 9050 6100 50  0000 L CNN
+F 1 "500/2W" V 8850 6000 50  0000 L CNN
+F 2 "" V 8880 6150 50  0001 C CNN
+F 3 "~" H 8950 6150 50  0001 C CNN
+	1    8950 6150
+	0    1    1    0
+$EndComp
+$Comp
+L Connector:Conn_Coaxial_Power J?
+U 1 1 641727E8
+P 9750 6450
+F 0 "J?" H 9950 6400 50  0000 C CNN
+F 1 "Sensor" H 9950 6500 50  0000 C CNN
+F 2 "" H 9750 6400 50  0001 C CNN
+F 3 "~" H 9750 6400 50  0001 C CNN
+	1    9750 6450
+	1    0    0    1
+$EndComp
+$Comp
+L Connector:Conn_Coaxial_Power J?
+U 1 1 641859E8
+P 8250 6450
+F 0 "J?" H 8050 6400 50  0000 C CNN
+F 1 "24VDC" H 8050 6500 50  0000 C CNN
+F 2 "" H 8250 6400 50  0001 C CNN
+F 3 "~" H 8250 6400 50  0001 C CNN
+	1    8250 6450
+	1    0    0    1
+$EndComp
+$Comp
+L Device:Fuse_Small F?
+U 1 1 642381A4
+P 8950 6550
+F 0 "F?" H 8950 6450 50  0000 C CNN
+F 1 "1A" H 8950 6644 50  0000 C CNN
+F 2 "" H 8950 6550 50  0001 C CNN
+F 3 "~" H 8950 6550 50  0001 C CNN
+	1    8950 6550
+	1    0    0    -1
+$EndComp
+Wire Wire Line
+	8250 6250 8250 6150
+Wire Wire Line
+	8250 5300 8450 5300
+Wire Wire Line
+	8800 6150 8250 6150
+Connection ~ 8250 6150
+Wire Wire Line
+	8250 6150 8250 5300
+Wire Wire Line
+	9750 6250 9750 6150
+Wire Wire Line
+	9750 6150 9350 6150
+Wire Wire Line
+	9350 5800 9350 6150
+Connection ~ 9350 6150
+Wire Wire Line
+	9350 6150 9100 6150
+Wire Wire Line
+	8250 6550 8850 6550
+Wire Wire Line
+	9050 6550 9750 6550
+Wire Wire Line
+	1900 6800 2500 6800
+Connection ~ 2500 6800
+Wire Wire Line
+	1900 6400 2050 6400
+Wire Wire Line
+	2250 6400 2500 6400
+Text Notes 8300 6350 0    50   ~ 0
+Phono
+Text Notes 9400 6350 0    50   ~ 0
+Phono
+Text Notes 1950 6700 0    50   ~ 0
+5.5x2.1
 $EndSCHEMATC

Commit message: v0.8 reconfigure manual override; updated layout for clarity
Parts:
- removed J?: Override, symbol Connector:Conn_01x03_Male
- removed SW?: Manual Override, symbol Switch:SW_SPDT
- removed SW?: SW_DPDT_x2, symbol Switch:SW_SPDT
- added J4: Override, symbol Connector:Conn_01x04_Male
- added R1: 270, symbol Device:R
- added SW1: Override, symbol Switch:SW_Push
- F1, F2: renamed from F?; footprint (none) -> Fuse:Fuse_SunFuse-6HP
- K5: renamed from K?; value Open-Close Relays -> Direction Relays
- R9: renamed from R?; value 500/2W -> 250/2W
- gave numbers to parts that had none: 38
Connections:
- net labels added: -12V
- net labels removed: +12V
- wire segments 256 -> 238
- no-connect marks 10 -> 37
Other:
- note added: "(open)-OFF-(close)"
- note added: "SPECIAL NOTE:\nThe override sense\ncircuitry has been\nabandoned but the\ncomponents are still\npresent on the board."
- note removed: "-12V"
- note removed: "Override"
- note removed: "RPi"
- moved on the sheet: BT1, F1, F2, J11, J12, J14, J15, J3, J5, J6, J7, J8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
